File: AMS_Fuse_ver2/AMS_Fuse_ver2.kicad_pcb (KiCad board)
At the start: 2 copper layers, 43 x 79 mm, 12 parts, among them J1 Conn_01x06_Socket, J2 Conn_01x06_Socket

Commit message: 位置修正
Parts:
- moved J2 4.75 mm to (138.4, 92.0)
Changed lines of the file:
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@@
   )
   (footprint "Connector_JST:JST_XH_S6B-XH-A_1x06_P2.50mm_Horizontal" (layer "F.Cu")
-    (at 138.45 96.75 -90)
+    (at 138.45 92 -90)
     (descr "JST XH series connector, S6B-XH-A (http://www.jst-mfg.com/product/pdf/eng/eXH.pdf), generated with kicad-footprint-generator")
     (tags "connector JST XH horizontal")
