File: AMS_Temp_i2c_Isolation/AMS_Temp_i2c_Isolation.kicad_sch (KiCad schematic)
At the start: 36 parts, among them J1 Conn_01x10_Socket, J2 Conn_01x06_Pin, J3 Conn_01x06_Pin, U1 ADuM1250, U2 LD1117S50TR_SOT223, U3 ATmega328P-A, Y1 CSTCE16M0V53-R0

Commit message: 回路図作成
Parts:
- added C12, C13: C, symbol Device:C
- added D5: D_Schottky, symbol Device:D_Schottky
- added J4, J5, J6: Conn_01x04_Pin, symbol Connector:Conn_01x04_Pin
- D2: value LED -> LED_R
- D3: value LED -> LED_G
Connections:
- net SCL is gone; now on net SCL1: U3.28 (PC5)
- net SDA is gone; now on net SDA1: U3.27 (PC4)
- net +12V: now also C2.1, C3.1, D1.1 (K), L1.2, U2.3 (VI), J4.1 (Pin_1), J5.4 (Pin_4), J6.1 (Pin_1)
- net +5VA: now also C11.1, J1.3 (Pin_3), PS1.6 (+Vout), R1.1, R10.1, R11.1, R12.1, R13.1, R2.1, R5.1, R6.1, R8.1, R9.1, U1.1 (VDD1), C12.1
- net +5VD: now also C10.1, C4.1, D1.2 (A), R3.1, R4.1, U1.8 (VDD2), U2.2 (VO)
- net GND1: now also J1.1 (Pin_1), J1.2 (Pin_2)
- net GNDA: now also C11.2, C8.2, D2.1 (K), J2.2 (Pin_2), J2.4 (Pin_4), J2.6 (Pin_6), J3.2 (Pin_2), J3.4 (Pin_4), J3.6 (Pin_6), PS1.7 (-Vout), U1.4 (GND1), C13.1
- net GNDD: now also C1.2, C10.2, C2.2, C3.2, C4.2, PS1.1 (-Vin), U1.5 (GND2), U2.1 (GND), C13.2, J4.4 (Pin_4), J5.1 (Pin_1), J6.4 (Pin_4)
- net MISO: now also J1.10 (Pin_10)
- net MOSI: now also J1.9 (Pin_9)
- net RESET: now also C9.1, J1.7 (Pin_7), R5.2, U3.29 (~{RESET}/PC6)
- net SCK: now also J1.8 (Pin_8)
- net Sens5: now reaches U3.19 (ADC6)
- net Sens5: now also J3.3 (Pin_3), R12.2
- net AREF: now reaches U3.20 (AREF)
- net AREF: now also C8.1
- net Sens6: now reaches U3.22 (ADC7)
- net Sens6: now also J3.5 (Pin_5), R13.2
- net Sens1: now reaches R8.2, U3.23 (PC0)
- net Sens1: now also J2.1 (Pin_1)
- net Sens2: now reaches R9.2, U3.24 (PC1)
- net Sens2: now also J2.3 (Pin_3)
- net Sens3: now reaches R10.2, U3.25 (PC2)
- net Sens3: now also J2.5 (Pin_5)
- net Sens4: now reaches R11.2, U3.26 (PC3)
- net Sens4: now also J3.1 (Pin_1)
- net RXI: now reaches U3.30 (PD0)
- net RXI: now also J1.4 (Pin_4)
- net TXO: now reaches U3.31 (PD1)
- net TXO: now also J1.5 (Pin_5)
- net SCL1: now reaches R2.2
- net SCL1: now also U1.3 (SCL1)
- net at C1.1: now also L1.1, D5.2 (A)
- net SDA1: now reaches U1.2 (SDA1)
- net SDA1: now also R1.2
- net SCL2: now reaches U1.6 (SCL2)
- net SCL2: now also R4.2, J4.3 (Pin_3), J5.2 (Pin_2), J6.3 (Pin_3)
- net SDA2: now reaches U1.7 (SDA2)
- net SDA2: now also R3.2, J4.2 (Pin_2), J5.3 (Pin_3), J6.2 (Pin_2)
- net at PS1.2 (+Vin): now also C12.2, D5.1 (K)
- net at R6.2: now also D2.2 (A)
- net DTR: now reaches J1.6 (Pin_6)
- net DTR: now also C9.2
Other:
- moved on the sheet: C1, C10, C11, C2, C3, C4, C8, C9, D1, D2, D3, J2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

Commit message: 温度監視回路図作成
Parts:
- removed D5: D_Schottky, symbol Device:D_Schottky
- removed J5: Conn_01x04_Pin, symbol Connector:Conn_01x04_Pin
- added D4: CUHS20S30, SamacSys_Parts:CUHS20S40H3F, symbol Device:D_Schottky
- C1, C2, C4: value C -> 10u; footprint (none) -> Capacitor_SMD:C_0805_2012Metric
- C10, C11, C3, C5, C6, C7, C8, C9: value C -> 0.1u; footprint (none) -> Capacitor_SMD:C_0603_1608Metric
- C12, C13: value C -> 220pF/3kV; footprint (none) -> Capacitor_SMD:C_1812_4532Metric
- D1: value D_Schottky -> CUHS20S30; footprint (none) -> SamacSys_Parts:CUHS20S40H3F
- D2, D3: footprint (none) -> LED_SMD:LED_0603_1608Metric
- J1: footprint (none) -> Connector_PinSocket_2.54mm:PinSocket_1x10_P2.54mm_Vertical
- J2, J3: footprint (none) -> Connector_JST:JST_XH_S6B-XH-A_1x06_P2.50mm_Horizontal
- J4: footprint (none) -> Connector_JST:JST_XH_S4B-XH-A_1x04_P2.50mm_Horizontal
- J6: footprint (none) -> Connector_PinHeader_2.54mm:PinHeader_1x04_P2.54mm_Vertical
- L1: value L -> 10u; footprint (none) -> Inductor_SMD:L_Taiyo-Yuden_NR-10050_9.8x10.0mm
- R1, R2, R3, R4: value R -> 3.3k; footprint (none) -> Resistor_SMD:R_0603_1608Metric
- R10, R11, R12, R13, R5, R8, R9: value R -> 10k; footprint (none) -> Resistor_SMD:R_0805_2012Metric
- R6, R7: value R -> Opt; footprint (none) -> Resistor_SMD:R_0603_1608Metric
Connections:
- net GND1 is gone; now on net GNDA: J1.1 (Pin_1), J1.2 (Pin_2)
- net +12V: now also D4.2 (A); no longer C2.1, L1.2
- net at C1.1, L1.1: now also C12.2, PS1.2 (+Vin)
- new net: C2.1, D4.1 (K), L1.2
Other:
- note added: "Isolation"
- moved on the sheet: C1, C2, J3, J4, L1

Commit message: Complete AMS_Temp_Master Circuit Schematics and modify
Parts:
- C1, C2, C4: footprint Capacitor_SMD:C_0805_2012Metric -> Capacitor_SMD:C_0603_1608Metric
- R10, R11, R12, R13, R5, R8, R9: footprint Resistor_SMD:R_0805_2012Metric -> Resistor_SMD:R_0603_1608Metric
Changed lines of the file:
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@@
       (effects (font (size 1.27 1.27)) (justify left))
     )
-    (property "Footprint" "Capacitor_SMD:C_0805_2012Metric" (at 257.5052 96.52 0)
+    (property "Footprint" "Capacitor_SMD:C_0603_1608Metric" (at 257.5052 96.52 0)
       (effects (font (size 1.27 1.27)) hide)
     )
@@
       (effects (font (size 1.27 1.27)) (justify left))
     )
-    (property "Footprint" "Resistor_SMD:R_0805_2012Metric" (at 140.462 57.15 90)
+    (property "Footprint" "Resistor_SMD:R_0603_1608Metric" (at 140.462 57.15 90)
       (effects (font (size 1.27 1.27)) hide)
     )
@@
       (effects (font (size 1.27 1.27)) (justify left))
     )
-    (property "Footprint" "Capacitor_SMD:C_0805_2012Metric" (at 237.1852 58.42 0)
+    (property "Footprint" "Capacitor_SMD:C_0603_1608Metric" (at 237.1852 58.42 0)
       (effects (font (size 1.27 1.27)) hide)
     )
@@
       (effects (font (size 1.27 1.27)) (justify left))
     )
-    (property "Footprint" "Resistor_SMD:R_0805_2012Metric" (at 163.322 72.39 90)
+    (property "Footprint" "Resistor_SMD:R_0603_1608Metric" (at 163.322 72.39 90)
       (effects (font (size 1.27 1.27)) hide)
     )
@@
       (effects (font (size 1.27 1.27)) (justify left))
     )
-    (property "Footprint" "Capacitor_SMD:C_0805_2012Metric" (at 249.8852 58.42 0)
+    (property "Footprint" "Capacitor_SMD:C_0603_1608Metric" (at 249.8852 58.42 0)
       (effects (font (size 1.27 1.27)) hide)
     )
@@
       (effects (font (size 1.27 1.27)) (justify left))
     )
-    (property "Footprint" "Resistor_SMD:R_0805_2012Metric" (at 132.842 52.07 90)
+    (property "Footprint" "Resistor_SMD:R_0603_1608Metric" (at 132.842 52.07 90)
       (effects (font (size 1.27 1.27)) hide)
     )
@@
       (effects (font (size 1.27 1.27)) (justify left))
     )
-    (property "Footprint" "Resistor_SMD:R_0805_2012Metric" (at 94.742 104.14 90)
+    (property "Footprint" "Resistor_SMD:R_0603_1608Metric" (at 94.742 104.14 90)
       (effects (font (size 1.27 1.27)) hide)
     )
@@
       (effects (font (size 1.27 1.27)) (justify left))
     )
-    (property "Footprint" "Resistor_SMD:R_0805_2012Metric" (at 155.702 67.31 90)
+    (property "Footprint" "Resistor_SMD:R_0603_1608Metric" (at 155.702 67.31 90)
       (effects (font (size 1.27 1.27)) hide)
     )
@@
       (effects (font (size 1.27 1.27)) (justify left))
     )
-    (property "Footprint" "Resistor_SMD:R_0805_2012Metric" (at 148.082 62.23 90)
+    (property "Footprint" "Resistor_SMD:R_0603_1608Metric" (at 148.082 62.23 90)
       (effects (font (size 1.27 1.27)) hide)
     )
@@
       (effects (font (size 1.27 1.27)) (justify left))
     )
-    (property "Footprint" "Resistor_SMD:R_0805_2012Metric" (at 125.222 46.99 90)
-      (effects (font (size 1.27 1.27)) hide)
-    )
+    (property "Footprint" "Resistor_SMD:R_0603_1608Metric" (at 125.222 46.99 90)
+      (effects (font (size 1.27 1.27)) hide)
+    )

Commit message: 部品配置
Parts:
- removed J1: Conn_01x10_Socket, Connector_PinSocket_2.54mm:PinSocket_1x10_P2.54mm_Vertical, symbol Connector:Conn_01x10_Socket
- removed J2, J3: Conn_01x06_Pin, Connector_JST:JST_XH_S6B-XH-A_1x06_P2.50mm_Horizontal, symbol Connector:Conn_01x06_Pin
- added J1, J10, J2, J3, J8, J9: Conn_01x02_Pin, Connector_JST:JST_XH_S2B-XH-A_1x02_P2.50mm_Horizontal, symbol Connector:Conn_01x02_Pin
- added J5: Conn_01x10_Socket, Connector_PinSocket_2.54mm:PinSocket_1x10_P2.54mm_Vertical, symbol Connector:Conn_01x10_Socket
Connections:
- net +5VA: now also J5.3 (Pin_3)
- net DTR: now also J5.6 (Pin_6)
- net GNDA: now also J1.2 (Pin_2), J10.2 (Pin_2), J2.2 (Pin_2), J3.2 (Pin_2), J5.1 (Pin_1), J5.2 (Pin_2), J8.2 (Pin_2), J9.2 (Pin_2)
- net MISO: now also J5.10 (Pin_10)
- net MOSI: now also J5.9 (Pin_9)
- net RESET: now also J5.7 (Pin_7)
- net RXI: now also J5.4 (Pin_4)
- net SCK: now also J5.8 (Pin_8)
- net Sens1: now also J1.1 (Pin_1)
- net Sens2: now also J2.1 (Pin_1)
- net Sens3: now also J3.1 (Pin_1)
- net Sens4: now also J8.1 (Pin_1)
- net Sens5: now also J9.1 (Pin_1)
- net Sens6: now also J10.1 (Pin_1)
- net TXO: now also J5.5 (Pin_5)

Commit message: 部品配置
Connections:
- net +Vin: now reaches C1.1, C12.2, L1.1, PS1.2 (+Vin)
- net _+Vin: now reaches C2.1, D4.1 (K), L1.2
Changed lines of the file:
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@@
   (junction (at 256.54 88.9) (diameter 0) (color 0 0 0 0)
-  )
-  (junction (at 233.68 50.8) (diameter 0) (color 0 0 0 0)
   )
   (junction (at 185.42 121.92) (diameter 0) (color 0 0 0 0)
@@
     (stroke (width 0) (type default))
   )
-  (wire (pts (xy 228.6 50.8) (xy 233.68 50.8))
-    (stroke (width 0) (type default))
-  )
   (wire (pts (xy 38.1 154.94) (xy 76.2 154.94))
     (stroke (width 0) (type default))
@@
     (stroke (width 0) (type default))
   )
-  (wire (pts (xy 233.68 50.8) (xy 236.22 50.8))
+  (wire (pts (xy 228.6 50.8) (xy 236.22 50.8))
     (stroke (width 0) (type default))
   )
@@
     (effects (font (size 1.27 1.27)) (justify left bottom))
   )
+  (label "_+Vin" (at 248.92 50.8 0) (fields_autoplaced)
+    (effects (font (size 1.27 1.27)) (justify left bottom))
+  )
   (label "Sens4" (at 129.54 96.52 0) (fields_autoplaced)
     (effects (font (size 1.27 1.27)) (justify left bottom))
@@
   )
   (label "AREF" (at 20.32 55.88 0) (fields_autoplaced)
+    (effects (font (size 1.27 1.27)) (justify left bottom))
+  )
+  (label "+Vin" (at 228.6 50.8 0) (fields_autoplaced)
     (effects (font (size 1.27 1.27)) (justify left bottom))
   )
@@
     )
   )
-  (symbol (lib_id "power:PWR_FLAG") (at 233.68 50.8 0) (unit 1)
+  (symbol (lib_id "power:PWR_FLAG") (at 236.22 50.8 0) (unit 1)
     (in_bom yes) (on_board yes) (dnp no) (fields_autoplaced)
-    (property "Reference" "#FLG03" (at 233.68 48.895 0)
-      (effects (font (size 1.27 1.27)) hide)
-    )
-    (property "Value" "PWR_FLAG" (at 233.68 45.72 0)
+    (property "Reference" "#FLG03" (at 236.22 48.895 0)
+      (effects (font (size 1.27 1.27)) hide)
+    )
+    (property "Value" "PWR_FLAG" (at 236.22 45.72 0)
       (effects (font (size 1.27 1.27)))
     )
-    (property "Footprint" "" (at 233.68 50.8 0)
-      (effects (font (size 1.27 1.27)) hide)
-    )
-    (property "Datasheet" "~" (at 233.68 50.8 0)
-      (effects (font (size 1.27 1.27)) hide)
-    )
+    (property "Footprint" "" (at 236.22 50.8 0)
+      (effects (font (size 1.27 1.27)) hide)
+    )
+    (property "Datasheet" "~" (at 236.22 50.8 0)
+      (effects (font (size 1.27 1.27)) hide)
+    )

Commit message: 修正とパターン完成
Parts:
- removed C12, C13: 220pF/3kV, Capacitor_SMD:C_1812_4532Metric, symbol Device:C
- R10, R11, R12, R13, R8, R9: footprint Resistor_SMD:R_0603_1608Metric -> Resistor_SMD:R_0805_2012Metric
Changed lines of the file:
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@@
   (junction (at 78.74 152.4) (diameter 0) (color 0 0 0 0)
   )
-  (junction (at 203.2 50.8) (diameter 0) (color 0 0 0 0)
-  )
   (junction (at 167.64 99.06) (diameter 0) (color 0 0 0 0)
   )
@@
   (junction (at 236.22 58.42) (diameter 0) (color 0 0 0 0)
   )
-  (junction (at 228.6 50.8) (diameter 0) (color 0 0 0 0)
-  )
   (junction (at 251.46 137.16) (diameter 0) (color 0 0 0 0)
   )
@@
   (junction (at 193.04 137.16) (diameter 0) (color 0 0 0 0)
   )
-  (junction (at 228.6 55.88) (diameter 0) (color 0 0 0 0)
-  )
   (junction (at 157.48 101.6) (diameter 0) (color 0 0 0 0)
   )
@@
   )
   (junction (at 238.76 132.08) (diameter 0) (color 0 0 0 0)
-  )
-  (junction (at 203.2 55.88) (diameter 0) (color 0 0 0 0)
   )
   (junction (at 266.7 50.8) (diameter 0) (color 0 0 0 0)
@@
     (stroke (width 0) (type default))
   )
-  (wire (pts (xy 212.09 38.1) (xy 203.2 38.1))
-    (stroke (width 0) (type default))
-  )
-  (wire (pts (xy 198.12 50.8) (xy 203.2 50.8))
+  (wire (pts (xy 198.12 50.8) (xy 205.74 50.8))
     (stroke (width 0) (type default))
   )
@@
     (stroke (width 0) (type default))
   )
-  (wire (pts (xy 198.12 55.88) (xy 203.2 55.88))
+  (wire (pts (xy 198.12 55.88) (xy 205.74 55.88))
     (stroke (width 0) (type default))
   )
@@
     (stroke (width 0) (type default))
   )
-  (wire (pts (xy 231.14 55.88) (xy 228.6 55.88))
+  (wire (pts (xy 226.06 55.88) (xy 231.14 55.88))
     (stroke (width 0) (type default))
   )
@@
     (stroke (width 0) (type default))
   )
-  (wire (pts (xy 203.2 68.58) (xy 203.2 55.88))
-    (stroke (width 0) (type default))
-  )
   (wire (pts (xy 167.64 99.06) (xy 167.64 91.44))
     (stroke (width 0) (type default))
@@
     (stroke (width 0) (type default))
   )
-  (wire (pts (xy 219.71 38.1) (xy 228.6 38.1))
-    (stroke (width 0) (type default))
-  )
   (wire (pts (xy 167.64 109.22) (xy 167.64 104.14))
     (stroke (width 0) (type default))
@@
     (stroke (width 0) (type default))
   )
-  (wire (pts (xy 203.2 50.8) (xy 205.74 50.8))
-    (stroke (width 0) (type default))
-  )
   (wire (pts (xy 124.46 101.6) (xy 157.48 101.6))
     (stroke (width 0) (type default))
@@
     (stroke (width 0) (type default))
   )
-  (wire (pts (xy 203.2 38.1) (xy 203.2 50.8))
-    (stroke (width 0) (type default))
-  )
   (wire (pts (xy 246.38 137.16) (xy 251.46 137.16))
     (stroke (width 0) (type default))
@@
     (stroke (width 0) (type default))
   )
-  (wire (pts (xy 212.09 68.58) (xy 203.2 68.58))
-    (stroke (width 0) (type default))
-  )
-  (wire (pts (xy 228.6 38.1) (xy 228.6 50.8))
-    (stroke (width 0) (type default))
-  )
   (wire (pts (xy 236.22 50.8) (xy 238.76 50.8))
     (stroke (width 0) (type default))
@@
     (stroke (width 0) (type default))
   )
-  (wire (pts (xy 203.2 55.88) (xy 205.74 55.88))
-    (stroke (width 0) (type default))
-  )
   (wire (pts (xy 38.1 152.4) (xy 78.74 152.4))
     (stroke (width 0) (type default))
@@
     (stroke (width 0) (type default))
   )
-  (wire (pts (xy 228.6 55.88) (xy 226.06 55.88))
-    (stroke (width 0) (type default))
-  )
   (wire (pts (xy 109.22 91.44) (xy 66.04 91.44))
     (stroke (width 0) (type default))
@@
     (stroke (width 0) (type default))
   )
-  (wire (pts (xy 228.6 50.8) (xy 236.22 50.8))
-    (stroke (width 0) (type default))
-  )
   (wire (pts (xy 248.92 88.9) (xy 256.54 88.9))
     (stroke (width 0) (type default))
@@
   )
   (wire (pts (xy 91.44 107.95) (xy 91.44 93.98))
-    (stroke (width 0) (type default))
-  )
-  (wire (pts (xy 219.71 68.58) (xy 228.6 68.58))
     (stroke (width 0) (type default))
   )
@@
     (stroke (width 0) (type default))
   )
-  (wire (pts (xy 228.6 68.58) (xy 228.6 55.88))
-    (stroke (width 0) (type default))
-  )
-  (wire (pts (xy 226.06 50.8) (xy 228.6 50.8))
+  (wire (pts (xy 226.06 50.8) (xy 236.22 50.8))
     (stroke (width 0) (type default))
   )
@@
       (effects (font (size 1.27 1.27)) (justify left))
     )
-    (property "Footprint" "Resistor_SMD:R_0603_1608Metric" (at 140.462 57.15 90)
+    (property "Footprint" "Resistor_SMD:R_0805_2012Metric" (at 140.462 57.15 90)
       (effects (font (size 1.27 1.27)) hide)
     )
@@
       (effects (font (size 1.27 1.27)) (justify left))
     )
-    (property "Footprint" "Resistor_SMD:R_0603_1608Metric" (at 163.322 72.39 90)
+    (property "Footprint" "Resistor_SMD:R_0805_2012Metric" (at 163.322 72.39 90)
       (effects (font (size 1.27 1.27)) hide)
     )
@@
         (path "/44c983c3-109e-4ba2-be45-c167f44ffda1"
           (reference "#PWR014") (unit 1)
-        )
-      )
-    )
-  )
-  (symbol (lib_id "Device:C") (at 215.9 68.58 90) (unit 1)
-    (in_bom yes) (on_board yes) (dnp no) (fields_autoplaced)
-    (property "Reference" "C13" (at 215.9 60.96 90)
-      (effects (font (size 1.27 1.27)))
-    )
-    (property "Value" "220pF/3kV" (at 215.9 63.5 90)
-      (effects (font (size 1.27 1.27)))
-    )
-    (property "Footprint" "Capacitor_SMD:C_1812_4532Metric" (at 219.71 67.6148 0)
-      (effects (font (size 1.27 1.27)) hide)
-    )
-    (property "Datasheet" "~" (at 215.9 68.58 0)
-      (effects (font (size 1.27 1.27)) hide)
-    )
-    (pin "1")
-    (pin "2")
-    (instances
-      (project "AMS_Temp_i2c_Isolation"
-        (path "/44c983c3-109e-4ba2-be45-c167f44ffda1"
-          (reference "C13") (unit 1)
         )
       )
@@
       (effects (font (size 1.27 1.27)) (justify left))
     )
-    (property "Footprint" "Resistor_SMD:R_0603_1608Metric" (at 132.842 52.07 90)
+    (property "Footprint" "Resistor_SMD:R_0805_2012Metric" (at 132.842 52.07 90)
       (effects (font (size 1.27 1.27)) hide)
     )
@@
       (effects (font (size 1.27 1.27)) (justify left))
     )
-    (property "Footprint" "Resistor_SMD:R_0603_1608Metric" (at 155.702 67.31 90)
+    (property "Footprint" "Resistor_SMD:R_0805_2012Metric" (at 155.702 67.31 90)
       (effects (font (size 1.27 1.27)) hide)
     )
@@
       (effects (font (size 1.27 1.27)) (justify left))
     )
-    (property "Footprint" "Resistor_SMD:R_0603_1608Metric" (at 148.082 62.23 90)
+    (property "Footprint" "Resistor_SMD:R_0805_2012Metric" (at 148.082 62.23 90)
       (effects (font (size 1.27 1.27)) hide)
     )
@@
     )
   )
-  (symbol (lib_id "Device:C") (at 215.9 38.1 90) (unit 1)
-    (in_bom yes) (on_board yes) (dnp no) (fields_autoplaced)
-    (property "Reference" "C12" (at 215.9 30.48 90)
-      (effects (font (size 1.27 1.27)))
-    )
-    (property "Value" "220pF/3kV" (at 215.9 33.02 90)
-      (effects (font (size 1.27 1.27)))
-    )
-    (property "Footprint" "Capacitor_SMD:C_1812_4532Metric" (at 219.71 37.1348 0)
-      (effects (font (size 1.27 1.27)) hide)
-    )
-    (property "Datasheet" "~" (at 215.9 38.1 0)
-      (effects (font (size 1.27 1.27)) hide)
-    )
-    (pin "1")
-    (pin "2")
-    (instances
-      (project "AMS_Temp_i2c_Isolation"
-        (path "/44c983c3-109e-4ba2-be45-c167f44ffda1"
-          (reference "C12") (unit 1)
-        )
-      )
-    )
-  )
   (symbol (lib_id "Device:R") (at 127 46.99 0) (unit 1)
     (in_bom yes) (on_board yes) (dnp no) (fields_autoplaced)
@@
       (effects (font (size 1.27 1.27)) (justify left))
     )
-    (property "Footprint" "Resistor_SMD:R_0603_1608Metric" (at 125.222 46.99 90)
-      (effects (font (size 1.27 1.27)) hide)
-    )
+    (property "Footprint" "Resistor_SMD:R_0805_2012Metric" (at 125.222 46.99 90)
+      (effects (font (size 1.27 1.27)) hide)
+    )
