File: AMS_Temp_Iso_ver2/AMS_Temp_Iso_ver2.kicad_pcb (KiCad board)
At the start: 2 copper layers, 70 x 102.5 mm, 75 parts, among them J1 Conn_01x02_Pin, J10 Conn_01x02_Pin, J11 Conn_01x02_Pin, J12 Conn_01x02_Pin, J13 Conn_01x10_Socket, J14 Conn_01x04_Pin, J15 Conn_01x04_Pin, J16 Conn_01x04_Pin, J17 Conn_01x04_Pin, J18 Conn_01x02_Pin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

Commit message: 残りはベタ修正
Parts:
- added ?: , , F.Cu at (141.5, 61.0)
- added ?: , , F.Cu at (136.5, 85.0)
- moved J16 39.4 mm to (137.0, 57.5), turned to 180 degrees
- moved R17 34.1 mm to (126.8, 86.5)
- moved R16 34.1 mm to (128.4, 86.5)
- moved C11 33.5 mm to (131.2, 89.0), turned to 180 degrees
- moved C12 33.3 mm to (142.1, 89.0), turned to 0 degrees
- moved U3 32.4 mm to (136.5, 90.9)
- moved C14 31.4 mm to (124.4, 83.4), turned to -90 degrees
- moved U4 29.9 mm to (121.0, 84.5)
- moved D4 29.3 mm to (121.5, 77.5)
- moved C13 28.0 mm to (120.3, 80.8), turned to 0 degrees
- moved J17 11.8 mm to (160.5, 70.0)
- moved C10 10.1 mm to (150.0, 66.5), turned to 0 degrees
- moved PS1 9.18 mm to (128.6, 73.9), turned to 0 degrees
- moved D3 8.36 mm to (124.0, 58.5), turned to 90 degrees
- moved R19 8.25 mm to (162.9, 76.0), turned to 90 degrees
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Connections:
- R1 pad 1: +5VA -> +5V
- R10 pad 1: +5VD -> +5V
- R11 pad 1: +5VD -> +5V
- R12 pad 1: +5VD -> +5V
- R13 pad 1: +5VD -> +5V
- R2 pad 1: +5VA -> +5V
- R3 pad 1: +5VA -> +5V
- R4 pad 1: +5VA -> +5V
- R5 pad 1: +5VA -> +5V
- R6 pad 1: +5VA -> +5V
- R8 pad 1: +5VD -> +5V
- R9 pad 1: +5VD -> +5V
- REF** pad 1: (no net) -> GND (x4)
- REF** pad 1: (no net) -> GND2 (x2)
- REF** pad 1: (no net) -> GND1 (x2)
Routing:
- net +5V: track 11.6 -> 179.9 mm
- net RESET: track 0.00 -> 59.3 mm, vias 0 -> 3
- net SCK: track 0.00 -> 57.9 mm, vias 0 -> 2
- net MISO: track 0.00 -> 57.1 mm, vias 0 -> 2
- net MOSI: track 0.00 -> 54.1 mm, vias 0 -> 2
- net RXI: track 0.00 -> 52.9 mm, vias 0 -> 3
- net TXO: track 0.00 -> 51.2 mm, vias 0 -> 3
- net SCL: track 0.00 -> 40.6 mm, vias 0 -> 2
- net SDA: track 0.00 -> 38.9 mm, vias 0 -> 2
- net +5VD: track 69.8 -> 31.9 mm, vias 3 -> 5
- net /Sens5: track 3.10 -> 39.3 mm, vias 0 -> 2
- net GND1: track 30.1 -> 65.2 mm, vias 0 -> 3
- net /Sens11: track 3.10 -> 34.5 mm, vias 0 -> 2
- net +5VA: track 89.4 -> 58.5 mm, vias 3 -> 4
- net /Sens6: track 3.10 -> 33.3 mm, vias 0 -> 2
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- added copper zone on B.Cu, net GND
- added copper zone on F.Cu, net GND
- added copper zone on B.Cu, net GND1
- added copper zone on F.Cu, net GND1
- added copper zone on B.Cu, net GND2
- added copper zone on F.Cu, net GND2

Commit message: pcb修正
Parts:
- moved D1 0.90 mm to (116.1, 123.2)
- moved D2 0.90 mm to (140.1, 123.2)
- moved R14 0.90 mm to (138.5, 123.2)
- moved R7 0.90 mm to (114.4, 123.2)
Routing:
- net GND1: track 65.2 -> 47.6 mm
- net GND: track 8.32 -> 10.9 mm, vias 1 -> 2
- net /SDA1: track 74.9 -> 77.4 mm
- net +12V: track 38.7 -> 37.4 mm
- net /SCL1: track 83.2 -> 84.2 mm
- net +5VA: track 58.5 -> 59.4 mm

Commit message: 修正
Routing:
- net +5V: track 179.6 -> 177.1 mm
- net GND: track 10.9 -> 11.6 mm
Other:
- board text added: "U1"
- board text added: "U2"

Commit message: パターン設計ほぼ完了
Parts:
- added REF**: BF@StampHole2.54, MyFootprints:BF@StampHole2.54, F.Cu at (98.8, 60.0)
- added REF**: BF@StampHole2.54, MyFootprints:BF@StampHole2.54, F.Cu at (171.2, 85.0)
- added REF**: BF@StampHole2.54, MyFootprints:BF@StampHole2.54, F.Cu at (155.0, 46.2)
- added REF**: BF@StampHole2.54, MyFootprints:BF@StampHole2.54, F.Cu at (135.0, 151.2)
- added REF**: BF@StampHole2.54, MyFootprints:BF@StampHole2.54, F.Cu at (135.0, 46.2)
- added REF**: BF@StampHole2.54, MyFootprints:BF@StampHole2.54, F.Cu at (155.0, 151.2)
- added REF**: BF@StampHole2.54, MyFootprints:BF@StampHole2.54, F.Cu at (98.8, 85.0)
- added REF**: BF@StampHole2.54, MyFootprints:BF@StampHole2.54, F.Cu at (171.2, 137.5)
- added REF**: BF@StampHole2.54, MyFootprints:BF@StampHole2.54, F.Cu at (171.2, 60.0)
- added REF**: BF@StampHole2.54, MyFootprints:BF@StampHole2.54, F.Cu at (171.2, 112.5)
- added REF**: BF@StampHole2.54, MyFootprints:BF@StampHole2.54, F.Cu at (115.0, 151.2)
- added REF**: BF@StampHole2.54, MyFootprints:BF@StampHole2.54, F.Cu at (115.0, 46.2)
- added REF**: BF@StampHole2.54, MyFootprints:BF@StampHole2.54, F.Cu at (98.8, 137.5)
- added REF**: BF@StampHole2.54, MyFootprints:BF@StampHole2.54, F.Cu at (98.8, 112.5)
- moved R18 3.58 mm to (164.5, 79.6)
- moved R19 3.58 mm to (162.9, 79.6)
- moved J17 3.40 mm to (160.5, 73.4)
- moved J18 3.22 mm to (161.2, 130.9), turned to 90 degrees
- moved J19 3.09 mm to (161.2, 134.8), turned to 90 degrees
- moved C10 2.19 mm to (152.1, 67.3), turned to 90 degrees
- moved ? 2.00 mm to (141.6, 63.0)
- moved J14 0.50 mm to (160.0, 124.5)
Routing:
- net GND1: track 47.6 -> 25.9 mm
- net GND2: track 22.7 -> 8.76 mm
- net GND: track 11.6 -> 19.0 mm
- net +5VA: track 59.4 -> 55.3 mm
- net +5VP: track 66.1 -> 62.4 mm
- net +5V: track 177.1 -> 173.6 mm
- net /SDA2: track 52.1 -> 48.6 mm
- net /SCL2: track 47.3 -> 44.3 mm
- net +5VD: track 32.2 -> 29.6 mm, vias 5 -> 4
- net /Sens11: track 34.6 -> 32.6 mm
- net /Sens12: track 29.0 -> 27.1 mm
- net SDA: track 38.9 -> 38.4 mm
- net SCL: track 40.6 -> 40.1 mm
Other:
- board size 70 x 102.5 mm -> 85 x 117.5 mm

Commit message: 完成、これで発注予定
Parts:
- added ?: , , F.Cu at (170.2, 153.2)
- added ?: , , F.Cu at (170.2, 43.4)
- added ?: , , F.Cu at (99.8, 40.6)
- added ?: , , F.Cu at (99.8, 45.1)
- added ?: , , F.Cu at (170.2, 154.2)
- added ?: , , F.Cu at (99.8, 44.2)
- added ?: , , F.Cu at (99.8, 41.5)
- added ?: , , F.Cu at (170.2, 41.5)
- added ?: , , F.Cu at (170.2, 44.2)
- added ?: , , F.Cu at (99.8, 156.8)
- added ?: , , F.Cu at (99.8, 152.3)
- added ?: , , F.Cu at (99.8, 155.9)
- added ?: , , F.Cu at (170.2, 155.9)
- added ?: , , F.Cu at (170.2, 155.1)
- added ?: , , F.Cu at (170.2, 152.3)
- added ?: , , F.Cu at (170.2, 42.5)
- added ?: , , F.Cu at (99.8, 43.4)
- added ?: , , F.Cu at (170.2, 45.1)
- added ?: , , F.Cu at (99.8, 42.5)
- added ?: , , F.Cu at (170.2, 40.6)
- added ?: , , F.Cu at (99.8, 155.1)
- added ?: , , F.Cu at (170.2, 156.8)
- added ?: , , F.Cu at (99.8, 153.2)
- added ?: , , F.Cu at (99.8, 154.2)
- moved C15 2.17 mm to (109.3, 126.7)
- moved R15 2.17 mm to (111.1, 126.5)
Routing:
- net /DTR: track 3.20 -> 5.53 mm
- net +5V: track 173.6 -> 175.1 mm
- net GND: track 19.0 -> 20.2 mm, vias 2 -> 150
- net GND2: vias 0 -> 49
- net GND1: vias 3 -> 58
Other:
- outline, holes or cut-outs redrawn
- board text added: "12V"
- board text added: "5V"
- board text added: "A0"
- board text added: "A1"
- board text added: "A2"
- board text added: "A3"
- board text added: "A6"
- board text added: "A7"
- board text added: "CTS"
- board text added: "DTR"
- board text added: "GND"
- board text added: "MISO"
- board text added: "MOSI"
- board text added: "RESET"
- board text added: "RXI"
- board text added: "SCK"
- board text added: "SCL"
- board text added: "SDA"
- board text added: "TXO"
- board text added: "VCC"
