File: AMS_Temp_Iso_ver2/AMS_Temp_Iso_ver2.kicad_sch (KiCad schematic)
At the start: 64 parts, among them J1 Conn_01x02_Pin, J10 Conn_01x02_Pin, J11 Conn_01x02_Pin, J12 Conn_01x02_Pin, J13 Conn_01x10_Socket, J14 Conn_01x04_Pin, J15 Conn_01x04_Pin, J16 Conn_01x04_Pin, J17 Conn_01x04_Pin, J18 Conn_01x02_Pin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

Commit message: 残りはベタ修正
Connections:
- net +5V: now also R1.1, R10.1, R11.1, R12.1, R13.1, R2.1, R3.1, R4.1, R5.1, R6.1, R8.1, R9.1
- net +5VA: no longer R1.1, R2.1, R3.1, R4.1, R5.1, R6.1
- net +5VD: no longer R10.1, R11.1, R12.1, R13.1, R8.1, R9.1
Changed lines of the file:
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@@
   (junction (at 124.46 119.38) (diameter 0) (color 0 0 0 0)
   )
-  (junction (at 259.08 68.58) (diameter 0) (color 0 0 0 0)
-  )
   (junction (at 114.3 109.22) (diameter 0) (color 0 0 0 0)
   )
-  (junction (at 121.92 68.58) (diameter 0) (color 0 0 0 0)
-  )
   (junction (at 50.8 30.48) (diameter 0) (color 0 0 0 0)
   )
@@
   (junction (at 91.44 68.58) (diameter 0) (color 0 0 0 0)
   )
+  (junction (at 121.92 68.58) (diameter 0) (color 0 0 0 0)
+  )
   (junction (at 261.62 119.38) (diameter 0) (color 0 0 0 0)
   )
@@
   (junction (at 243.84 137.16) (diameter 0) (color 0 0 0 0)
   )
+  (junction (at 259.08 68.58) (diameter 0) (color 0 0 0 0)
+  )
   (junction (at 106.68 68.58) (diameter 0) (color 0 0 0 0)
   )
@@
     )
   )
-  (symbol (lib_id "power:+5VA") (at 121.92 68.58 0) (unit 1)
-    (in_bom yes) (on_board yes) (dnp no) (fields_autoplaced)
-    (property "Reference" "#PWR016" (at 121.92 72.39 0)
-      (effects (font (size 1.27 1.27)) hide)
-    )
-    (property "Value" "+5VA" (at 121.92 63.5 0)
-      (effects (font (size 1.27 1.27)))
-    )
-    (property "Footprint" "" (at 121.92 68.58 0)
-      (effects (font (size 1.27 1.27)) hide)
-    )
-    (property "Datasheet" "" (at 121.92 68.58 0)
-      (effects (font (size 1.27 1.27)) hide)
-    )
-    (pin "1")
-    (instances
-      (project "AMS_Temp_Iso_ver2"
-        (path "/80f5cc61-e4d3-41fb-be7d-36378cd0c526"
-          (reference "#PWR016") (unit 1)
-        )
-      )
-    )
-  )
   (symbol (lib_id "Connector:Conn_01x02_Pin") (at 132.08 116.84 0) (mirror y) (unit 1)
     (in_bom yes) (on_board yes) (dnp no) (fields_autoplaced)
@@
     )
   )
-  (symbol (lib_id "power:+5VD") (at 259.08 68.58 0) (unit 1)
-    (in_bom yes) (on_board yes) (dnp no) (fields_autoplaced)
-    (property "Reference" "#PWR021" (at 259.08 72.39 0)
-      (effects (font (size 1.27 1.27)) hide)
-    )
-    (property "Value" "+5VD" (at 259.08 63.5 0)
-      (effects (font (size 1.27 1.27)))
-    )
-    (property "Footprint" "" (at 259.08 68.58 0)
-      (effects (font (size 1.27 1.27)) hide)
-    )
-    (property "Datasheet" "" (at 259.08 68.58 0)
-      (effects (font (size 1.27 1.27)) hide)
-    )
-    (pin "1")
-    (instances
-      (project "AMS_Temp_Iso_ver2"
-        (path "/80f5cc61-e4d3-41fb-be7d-36378cd0c526"
-          (reference "#PWR021") (unit 1)
-        )
-      )
-    )
-  )
   (symbol (lib_id "Device:C") (at 38.1 26.67 0) (unit 1)
     (in_bom yes) (on_board yes) (dnp no) (fields_autoplaced)
@@
     )
   )
+  (symbol (lib_id "power:+5V") (at 121.92 68.58 0) (unit 1)
+    (in_bom yes) (on_board yes) (dnp no) (fields_autoplaced)
+    (property "Reference" "#PWR021" (at 121.92 72.39 0)
+      (effects (font (size 1.27 1.27)) hide)
+    )
+    (property "Value" "+5V" (at 121.92 63.5 0)
+      (effects (font (size 1.27 1.27)))
+    )
+    (property "Footprint" "" (at 121.92 68.58 0)
+      (effects (font (size 1.27 1.27)) hide)
+    )
+    (property "Datasheet" "" (at 121.92 68.58 0)
+      (effects (font (size 1.27 1.27)) hide)
+    )
+    (pin "1")
+    (instances
+      (project "AMS_Temp_Iso_ver2"
+        (path "/80f5cc61-e4d3-41fb-be7d-36378cd0c526"
+          (reference "#PWR021") (unit 1)
+        )
+      )
+    )
+  )
   (symbol (lib_id "Device:R") (at 251.46 72.39 0) (unit 1)
     (in_bom yes) (on_board yes) (dnp no) (fields_autoplaced)
@@
         )
       )
+    )
+  )
+  (symbol (lib_id "power:+5V") (at 259.08 68.58 0) (unit 1)
+    (in_bom yes) (on_board yes) (dnp no) (fields_autoplaced)
+    (property "Reference" "#PWR016" (at 259.08 72.39 0)
+      (effects (font (size 1.27 1.27)) hide)
+    )
+    (property "Value" "+5V" (at 259.08 63.5 0)
+      (effects (font (size 1.27 1.27)))
+    )
+    (property "Footprint" "" (at 259.08 68.58 0)
+      (effects (font (size 1.27 1.27)) hide)
+    )
+    (property "Datasheet" "" (at 259.08 68.58 0)
+      (effects (font (size 1.27 1.27)) hide)
+    )
+    (pin "1")
+    (instances
+      (project "AMS_Temp_Iso_ver2"
+        (path "/80f5cc61-e4d3-41fb-be7d-36378cd0c526"
+          (reference "#PWR016") (unit 1)
+        )
+      )
