File: ECUShield_MEGA/ECUShield_MEGA.kicad_sch (KiCad schematic)
At the start: 23 parts, among them J1 Power, J10 Conn_01x02_Pin, J11 Conn_01x02_Pin, J12 Conn_01x03_Pin, J13 Conn_01x03_Pin, J3 Analog, J4 PWM, J5 Analog, J6 Communication, J7 Conn_01x02_Pin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

Commit message: 更新
Parts:
- added R5, R6: 10k, Resistor_SMD:R_0805_2012Metric, symbol Device:R
- added R7, R8: 3.3k, Resistor_SMD:R_0603_1608Metric, symbol Device:R
Connections:
- net +5V: now also R7.1, R8.1
- net SCL/21: now also J9.2 (Pin_2), R8.2
- net SDA/20: now also J9.1 (Pin_1), R7.2
Other:
- moved on the sheet: J8, J9
