File: ECUShield_MEGA_ver1/ECUShield_MEGA_ver1.kicad_pcb (KiCad board)
At the start: 2 copper layers, 101.6 x 53.3 mm, 34 parts, among them J1 Power, J10 Conn_01x02_Pin, J11 Conn_01x02_Pin, J12 Conn_01x02_Pin, J13 Conn_01x03_Pin, J14 Conn_01x03_Pin, J2 PWM, J3 Analog, J4 PWM, J5 Analog, J6 Communication, J7 Conn_02x03_Odd_Even, J7 Digital, J8 Conn_01x02_Pin, J9 Conn_01x02_Pin, K1 G5Q-1, K2 G5Q-1, Q1 2SC1815, Q2 2SC1815, Q3 2SC1815

Commit message: 回路図作成, パターン作成途中
Parts:
- removed the J10 at (49.4, 47.5)
- removed the J11 at (49.4, 55.2)
- removed the J12 at (49.4, 63.0)
- removed the J8 at (49.4, 31.9)
- removed the J9 at (49.4, 39.6)
- added C1: 0.1u, Capacitor_SMD:C_0603_1608Metric, F.Cu at (178.9, 68.3)
- added C2: 0.1u, Capacitor_SMD:C_0603_1608Metric, F.Cu at (182.1, 54.9)
- added D3: 1S953, Diode_THT:D_DO-35_SOD27_P7.62mm_Horizontal, F.Cu at (138.8, 70.3)
- added J15: Conn_01x02_Pin, Connector_JST:JST_XH_B2B-XH-A_1x02_P2.50mm_Vertical, F.Cu at (105.5, 83.4)
- added J16: Conn_01x02_Pin, Connector_JST:JST_XH_B2B-XH-A_1x02_P2.50mm_Vertical, F.Cu at (105.5, 92.2)
- added J17: Conn_01x02_Pin, Connector_JST:JST_XH_B2B-XH-A_1x02_P2.50mm_Vertical, F.Cu at (148.6, 40.8)
- added J18: Conn_01x02_Pin, Connector_JST:JST_XH_B2B-XH-A_1x02_P2.50mm_Vertical, F.Cu at (152.6, 68.0)
- added J19: Conn_01x02_Pin, Connector_JST:JST_XH_B2B-XH-A_1x02_P2.50mm_Vertical, F.Cu at (148.1, 58.2)
- added J2: Conn_01x02_Pin, Connector_JST:JST_XH_B2B-XH-A_1x02_P2.50mm_Vertical, F.Cu at (148.2, 90.5)
- added J20: Conn_01x02_Pin, Connector_JST:JST_XH_B2B-XH-A_1x02_P2.50mm_Vertical, F.Cu at (180.8, 76.5)
- added J3: Conn_01x02_Pin, Connector_JST:JST_XH_B2B-XH-A_1x02_P2.50mm_Vertical, F.Cu at (138.8, 63.6)
- added J4: Conn_01x03_Pin, Connector_JST:JST_XH_B3B-XH-A_1x03_P2.50mm_Vertical, F.Cu at (155.5, 83.5)
- added J5: Conn_01x03_Pin, Connector_JST:JST_XH_B3B-XH-A_1x03_P2.50mm_Vertical, F.Cu at (166.5, 83.5)
- added J6: Conn_01x02_Pin, Connector_JST:JST_XH_B2B-XH-A_1x02_P2.50mm_Vertical, F.Cu at (177.8, 88.5)
- added Q4: MTN2306AN3, Package_TO_SOT_SMD:TSOT-23, F.Cu at (151.4, 35.2)
- added R10: 3.3k, Resistor_SMD:R_0603_1608Metric, F.Cu at (110.7, 49.2)
- added R11: 10k, Resistor_SMD:R_0805_2012Metric, F.Cu at (146.9, 65.4)
- added R12: 10k, Resistor_SMD:R_0805_2012Metric, F.Cu at (146.3, 53.3)
- added R13: 3.3k, Resistor_SMD:R_0603_1608Metric, F.Cu at (103.7, 50.6)
- added R7: 1M, Resistor_SMD:R_0603_1608Metric, F.Cu at (120.6, 55.6)
- added R8: 1M, Resistor_SMD:R_0603_1608Metric, F.Cu at (128.0, 55.6)
- added R9: 1M, Resistor_SMD:R_0603_1608Metric, F.Cu at (151.4, 31.1)
- added U1: MCP2515-xST, Package_SO:TSSOP-20_4.4x6.5mm_P0.65mm, F.Cu at (174.6, 64.6)
- added U2: MCP2551-I-SN, Package_SO:SOIC-8_3.9x4.9mm_P1.27mm, F.Cu at (182.0, 59.5)
- added Y1: CSTCE16M0V53-R0, SamacSys_Parts:CSTCE16M0V53R0, F.Cu at (172.6, 58.4)
- D1: value 1S953 -> NUP2105L; footprint Diode_THT:D_DO-35_SOD27_P7.62mm_Horizontal -> Package_TO_SOT_SMD:SOT-23
- J13, J14: value Conn_01x03_Pin -> Conn_01x02_Pin; footprint Connector_JST:JST_XH_S3B-XH-A_1x03_P2.50mm_Horizontal -> Connector_JST:JST_XH_B2B-XH-A_1x02_P2.50mm_Vertical
- Q1, Q2, Q3: value 2SC1815 -> MTN2306AN3; footprint Package_TO_SOT_THT:TO-92L_Inline_Wide -> Package_TO_SOT_SMD:TSOT-23
- R2: value 10k -> 1M; footprint Resistor_SMD:R_0805_2012Metric -> Resistor_SMD:R_0603_1608Metric
- R5: value 10k -> 15k; footprint Resistor_SMD:R_0805_2012Metric -> Resistor_SMD:R_0603_1608Metric
- R6: value 10k -> 120; footprint Resistor_SMD:R_0805_2012Metric -> Resistor_SMD:R_0603_1608Metric
- moved R1 111.2 mm to (178.1, 82.9)
- moved R5 107.3 mm to (185.6, 62.8), turned to -90 degrees
- moved R6 104.8 mm to (182.0, 70.0), turned to 180 degrees
- moved D1 103.9 mm to (182.0, 66.0), turned to -90 degrees
- moved R4 102.6 mm to (177.7, 71.1)
- moved Q1 79.5 mm to (136.4, 56.8), turned to 180 degrees
- moved K2 77.2 mm to (131.2, 75.1), turned to -90 degrees
- moved Q3 75.6 mm to (131.4, 55.5)
- moved Q2 67.8 mm to (124.4, 55.5)
- moved K1 66.8 mm to (117.9, 67.9), turned to -90 degrees
- moved R2 64.9 mm to (140.7, 56.8), turned to 90 degrees
- moved R3 58.2 mm to (136.0, 52.7), turned to 180 degrees
- moved D2 47.2 mm to (125.6, 62.3), turned to 180 degrees
- moved J13 40.3 mm to (107.3, 56.5), turned to 180 degrees
- moved J14 31.8 mm to (105.5, 74.6)
- renumbered J7 to J1, J2 to J10, J4 to J11, J6 to J12, J1 to J7, J3 to J8, J5 to J9
Connections:
- net +3V3 renamed +3.3V
- net /~{RESET} renamed /RESET
- D1 pad 1: unconnected-(D1-K-Pad1) -> /CANH
- D1 pad 2: unconnected-(D1-A-Pad2) -> /CANL
- D2 pad 1: unconnected-(D2-K-Pad1) -> SHUTDOWN_CIRCUIT
- D2 pad 2: unconnected-(D2-A-Pad2) -> Net-(D2-A)
- J1 pad 1: unconnected-(J7-Pin_1-Pad1) (its old number) -> /MISO_A
- J1 pad 3: unconnected-(J7-Pin_3-Pad3) -> /SCK_A
- J1 pad 4: unconnected-(J7-Pin_4-Pad4) -> /MOSI_A
- J1 pad 6: unconnected-(J7-Pin_6-Pad6) -> GND
- J10 pad 9: /*9/CS -> /*9/CS_A
- J11 pad 6: /*2 -> /*2/INT_A
- J12 pad 7: /SDA/20 -> unconnected-(J12-Pin_7-Pad7)
- J12 pad 8: /SCL/21 -> unconnected-(J12-Pin_8-Pad8)
- J13 pad 1: unconnected-(J13-Pin_1-Pad1) -> /SDA/20
- J13 pad 2: unconnected-(J13-Pin_2-Pad2) -> /SCL/21
- J14 pad 1: unconnected-(J14-Pin_1-Pad1) -> GND
- J14 pad 2: unconnected-(J14-Pin_2-Pad2) -> /PRECHARGE
- K1 pad 1: unconnected-(K1-Pad1) -> Net-(D2-A)
- K1 pad 2: unconnected-(K1-Pad2) -> SHUTDOWN_CIRCUIT
- K1 pad 3: unconnected-(K1-Pad3) -> /AIR+
- K1 pad 4: unconnected-(K1-Pad4) -> /PRECHARGE
- K1 pad 5: unconnected-(K1-Pad5) -> SHUTDOWN_CIRCUIT
- K2 pad 1: unconnected-(K2-Pad1) -> Net-(D3-A)
- K2 pad 2: unconnected-(K2-Pad2) -> SHUTDOWN_CIRCUIT
- K2 pad 3: unconnected-(K2-Pad3) -> /AIR-
- K2 pad 5: unconnected-(K2-Pad5) -> SHUTDOWN_CIRCUIT
- Q1 pad 1: unconnected-(Q1-E-Pad1) -> SHUTDOWN_CIRCUIT
- Q1 pad 2: unconnected-(Q1-C-Pad2) -> GND
- Q1 pad 3: unconnected-(Q1-B-Pad3) -> /*11
- Q2 pad 1: unconnected-(Q2-E-Pad1) -> /*13
- Q2 pad 2: unconnected-(Q2-C-Pad2) -> GND
- Q2 pad 3: unconnected-(Q2-B-Pad3) -> Net-(D2-A)
- Q3 pad 1: unconnected-(Q3-E-Pad1) -> /*12
- Q3 pad 2: unconnected-(Q3-C-Pad2) -> GND
- Q3 pad 3: unconnected-(Q3-B-Pad3) -> Net-(D3-A)
- R1 pad 1: unconnected-(R1-Pad1) -> +5V
- R1 pad 2: unconnected-(R1-Pad2) -> /A2
- R2 pad 1: unconnected-(R2-Pad1) -> SHUTDOWN_CIRCUIT
- R2 pad 2: unconnected-(R2-Pad2) -> GND
- R3 pad 1: unconnected-(R3-Pad1) -> +5V
- R3 pad 2: unconnected-(R3-Pad2) -> /*11
- R4 pad 1: unconnected-(R4-Pad1) -> +5V
- R4 pad 2: unconnected-(R4-Pad2) -> Net-(U1-~{RESET})
- R5 pad 1: unconnected-(R5-Pad1) -> Net-(U2-Rs)
- R5 pad 2: unconnected-(R5-Pad2) -> GND
- R6 pad 1: unconnected-(R6-Pad1) -> /CANH
- R6 pad 2: unconnected-(R6-Pad2) -> /CANL

Commit message: 基板配置まで
Parts:
- removed the J7 at (194.0, 92.4)
- moved J16 91.6 mm to (197.0, 89.2), turned to 90 degrees
- moved J14 84.3 mm to (188.5, 89.2), turned to 90 degrees
- moved J15 74.8 mm to (180.0, 89.2), turned to 90 degrees
- moved J20 62.3 mm to (118.5, 78.2), turned to 90 degrees
- moved K2 58.5 mm to (188.2, 62.1)
- moved D3 58.5 mm to (195.8, 57.4)
- moved K1 56.6 mm to (174.2, 62.1)
- moved D2 56.4 mm to (181.8, 57.4)
- moved R8 55.7 mm to (183.7, 54.1)
- moved R6 55.5 mm to (126.8, 75.9), turned to 90 degrees
- moved Q3 55.5 mm to (186.9, 54.2)
- moved R5 54.5 mm to (133.7, 79.6), turned to 180 degrees
- moved D1 52.5 mm to (130.5, 76.0), turned to 180 degrees
- moved U2 48.0 mm to (137.0, 76.0), turned to 180 degrees
- moved R7 47.0 mm to (167.6, 54.9)
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Connections:
- J18 pad 1: /*10 -> /*12
- J19 pad 1: /*8 -> /*11
- J20 pad 1: /CANL -> /CANH
- J20 pad 2: /CANH -> /CANL
- Q1 pad 3: /*11 -> /*10
- Q2 pad 1: /*13 -> /*4
- Q3 pad 1: /*12 -> /*3
- Q4 pad 1: /*7 -> /*13
- R11 pad 1: /*10 -> /*12
- R12 pad 1: /*8 -> /*11
- R3 pad 2: /*11 -> /*10
- R7 pad 1: /*13 -> /*4
- R8 pad 1: /*12 -> /*3
- R9 pad 1: /*7 -> /*13
Other:
- board text added: "A0"
- board text added: "A1"
- board text added: "A10"
- board text added: "A11"
- board text added: "A12"
- board text added: "A13"
- board text added: "A14"
- board text added: "A15"
- board text added: "A2"
- board text added: "A3"
- board text added: "A4"
- board text added: "A5"
- board text added: "A6"
- board text added: "A7"
- board text added: "A8"
- board text added: "A9"

Commit message: パターン設計途中
Parts:
- moved Q4 2.83 mm to (121.0, 59.0)
- moved R9 2.83 mm to (121.1, 55.8)
- moved J13 2.50 mm to (110.0, 58.2)
- moved R11 2.24 mm to (129.0, 56.0)
- moved R12 2.24 mm to (129.0, 61.0)
- moved J17 2.00 mm to (110.0, 69.2)
- moved J18 2.00 mm to (118.5, 69.2)
- moved J19 2.00 mm to (127.0, 69.2)
- moved J20 2.00 mm to (118.5, 80.2)
- moved R1 0.24 mm to (166.5, 88.3)
Connections:
- net Net-(D2-A) renamed /COIL1
- net Net-(D3-A) renamed /COIL2
Routing:
- net +5V: track 0.00 -> 132.1 mm, vias 0 -> 2
- net SHUTDOWN_CIRCUIT: track 0.00 -> 99.8 mm, vias 0 -> 1
- net +12V: track 0.00 -> 63.0 mm, vias 0 -> 1
- net /*3: track 0.00 -> 32.7 mm, vias 0 -> 1
- net /*2/INT_A: track 0.00 -> 30.7 mm, vias 0 -> 2
- net /*9/CS_A: track 0.00 -> 29.8 mm
- net /*12: track 0.00 -> 28.5 mm
- net /*11: track 0.00 -> 24.2 mm
- net /MOSI_A: track 0.00 -> 23.6 mm
- net /TXCAN: track 0.00 -> 22.9 mm
- net /SDA/20: track 0.00 -> 22.6 mm
- net /A2: track 0.00 -> 20.7 mm
- net /SCL/21: track 0.00 -> 20.3 mm
- net /*4: track 0.00 -> 20.2 mm, vias 0 -> 1
- net /A1: track 0.00 -> 18.4 mm
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Other:
- board text added: "+3.3V"
- board text added: "+5V"
- board text added: "0"
- board text added: "1"
- board text added: "10"
- board text added: "11"
- board text added: "12"
- board text added: "13"
- board text added: "14"
- board text added: "15"
- board text added: "16"
- board text added: "17"
- board text added: "18"
- board text added: "19"
- board text added: "2"
- board text added: "20"
- board text added: "21"
- board text added: "3"
- board text added: "4"
- board text added: "5"
- board text added: "6"
- board text added: "7"
- board text added: "8"
- board text added: "9"
- board text added: "AREF"
- board text added: "GND"
- board text added: "IOREF"
- board text added: "RESET"
- board text added: "Vin"

Commit message: パターン作成途中
Parts:
- moved R1 8.35 mm to (159.0, 92.0), turned to 0 degrees
- moved R4 4.74 mm to (154.9, 66.1), turned to 0 degrees
- moved R6 4.00 mm to (123.8, 78.6)
- moved D1 3.43 mm to (127.1, 76.7)
- moved R5 3.43 mm to (130.3, 80.2)
- moved U2 3.43 mm to (133.6, 76.6)
- moved C2 3.43 mm to (138.9, 76.0)
- moved U1 2.63 mm to (151.1, 72.3)
- moved Y1 2.63 mm to (144.9, 74.3)
- moved C1 2.63 mm to (154.8, 68.0)
- moved Q1 1.36 mm to (136.3, 55.0)
- moved R2 1.36 mm to (136.2, 58.2)
- moved R3 1.24 mm to (133.5, 54.6)
- moved J5 1.00 mm to (161.5, 86.5)
Routing:
- net +5V: track 132.1 -> 150.1 mm
- net /MOSI_A: track 23.6 -> 13.2 mm, vias 0 -> 1
- net /*9/CS_A: track 29.8 -> 39.5 mm
- net Net-(U1-~{RESET}): track 3.64 -> 7.93 mm
- net /CANH: track 17.7 -> 14.5 mm
- net /CANL: track 17.3 -> 14.4 mm
- net /MISO_A: track 7.74 -> 10.4 mm
- net /SCK_A: track 7.98 -> 10.1 mm
- net SHUTDOWN_CIRCUIT: track 99.8 -> 101.7 mm
- net /A2: track 20.7 -> 22.1 mm
- net /A1: track 18.4 -> 19.7 mm
- net /*10: track 8.58 -> 7.42 mm
- net +12V: track 63.0 -> 61.9 mm, vias 1 -> 2
- net /*4: track 20.2 -> 19.2 mm
- net /RXCAN: track 15.0 -> 14.1 mm
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
Commit message: update
Routing:
- net GND: track 0.00 -> 11.6 mm, vias 0 -> 128
- net /A2: track 22.1 -> 21.6 mm
- added copper zone on B.Cu, net GND
- added copper zone on F.Cu, net GND
Other:
- board text added: "AIR+"
- board text added: "AIR-"
- board text added: "Accel1"
- board text added: "Accel2"
- board text added: "Brake"
- board text added: "CANH"
- board text added: "CANL"
- board text added: "Power"
- board text added: "Precharge"
- board text added: "Ready to Drive LED"
- board text added: "Ready to Drive SW"
- board text added: "SCL"
- board text added: "SDA"
- board text added: "Shutdown Circuit"
- board text added: "Shutdown SW"

Commit message: finish, ver1
Routing:
- net GND: vias 128 -> 130

Commit message: modify, finish, ver3
Connections:
- D2 pad 1: SHUTDOWN_CIRCUIT -> +12V
- D3 pad 1: SHUTDOWN_CIRCUIT -> +12V
- K1 pad 5: SHUTDOWN_CIRCUIT -> +12V
- K2 pad 5: SHUTDOWN_CIRCUIT -> +12V
Routing:
- net +12V: track 61.6 -> 148.1 mm, vias 2 -> 4
- net SHUTDOWN_CIRCUIT: track 101.7 -> 64.5 mm
- net /A0: track 17.2 -> 18.3 mm
- net GND: vias 130 -> 139
