File: ECUShield_MEGA_ver1/ECUShield_MEGA_ver1.kicad_sch (KiCad schematic)
At the start: 42 parts, among them J1 Power, J10 Conn_01x02_Pin, J11 Conn_01x02_Pin, J12 Conn_01x02_Pin, J13 Conn_01x03_Pin, J14 Conn_01x03_Pin, J15 Conn_01x02_Pin, J16 Conn_01x02_Pin, J17 Conn_01x02_Pin, J18 Conn_01x02_Pin, J2 PWM, J3 Analog, J4 PWM, J5 Analog, J6 Communication, J7 Conn_02x03_Odd_Even, J8 Conn_01x02_Pin, J9 Conn_01x02_Pin, K1 G5Q-1, K2 G5Q-1, Q1 2SC1815, Q2 2SC1815, Q3 2SC1815, U1 MCP2515-xST, U2 MCP2551-I-SN, Y1 CSTCE16M0V53-R0

Commit message: 回路図作成, パターン作成途中
Parts:
- removed Q1, Q2, Q3: 2SC1815, Package_TO_SOT_THT:TO-92L_Inline_Wide, symbol Transistor_BJT:2SC1815
- removed R4, R5, R6: 10k, Resistor_SMD:R_0805_2012Metric, symbol Device:R
- added J3, J6: Conn_01x02_Pin, Connector_JST:JST_XH_B2B-XH-A_1x02_P2.50mm_Vertical, symbol Connector:Conn_01x02_Pin
- added Q1, Q2, Q3, Q4: MTN2306AN3, Package_TO_SOT_SMD:TSOT-23, symbol Device:Q_NMOS_GSD
- added R10, R13: 3.3k, Resistor_SMD:R_0603_1608Metric, symbol Device:R
- added R2, R8, R9: 1M, Resistor_SMD:R_0603_1608Metric, symbol Device:R
- R7: renamed from R2; value 10k -> 1M; footprint Resistor_SMD:R_0805_2012Metric -> Resistor_SMD:R_0603_1608Metric
- renumbered D3 to D1, D1 to D2, D2 to D3, J7 to J1, J2 to J10, J4 to J11, J6 to J12, J9 to J13, J10 to J14, J11 to J15, J12 to J16, J15 to J17, J16 to J18, J17 to J19, J8 to J2, J18 to J20, J13 to J4, J14 to J5, J1 to J7, J3 to J8, J5 to J9, R10 to R11, R11 to R12, R9 to R4, R8 to R5, R7 to R6
Connections:
- net *10: now also J18.1 (Pin_1), R11.1
- net *11: now also R3.2, Q1.3 (D)
- net *12: now also Q3.1 (G), R8.1
- net *13: now also R7.1, Q2.1 (G)
- net *3: no longer J19.1 (Pin_1), R12.1
- net *4: no longer J18.1 (Pin_1), R11.1
- net *6: no longer R3.1
- net *7: now also Q4.1 (G), R9.1; no longer R1.1
- net *8: now also J19.1 (Pin_1), R12.1
- net +12V: no longer D2.1 (K), D3.1 (K), J14.2 (Pin_2), J15.2 (Pin_2), J16.2 (Pin_2), K1.5, K2.5
- net +5V: now also R1.1, R3.1, R10.1, R13.1
- net A2: now also R1.2, J6.1 (Pin_1)
- net GND: now also D1.3 (A), J1.6 (Pin_6), J14.1 (Pin_1), J15.1 (Pin_1), J16.1 (Pin_1), J3.2 (Pin_2), J6.2 (Pin_2), Q1.2 (S), Q2.2 (S), Q3.2 (S), Q4.2 (S), R2.2, R8.2, R9.2; no longer K1.2
- net SCL/21: now also R10.2; no longer J12.8 (Pin_8)
- net SDA/20: now also R13.2; no longer J12.7 (Pin_7)
- net CANH: now reaches D1.1 (K), J20.2 (Pin_2), R6.1, U2.7 (CANH)
- net CANL: now reaches D1.2 (K), J20.1 (Pin_1), R6.2, U2.6 (CANL)
- net at D3.2 (A), K2.1: now also Q3.3 (D)
- net SHUTDOWN_CIRCUIT: now reaches K2.2
- net SHUTDOWN_CIRCUIT: now also D2.1 (K), D3.1 (K), K1.2, K1.5, K2.5, J3.1 (Pin_1), Q1.1 (G), R2.1
- net AIR-: now reaches K2.3
- net AIR-: now also J16.2 (Pin_2); no longer J16.1 (Pin_1)
- net TXCAN: now reaches U1.1 (TXCAN), U2.1 (TXD)
- net RXCAN: now reaches U1.2 (RXCAN), U2.4 (RXD)
- net AIR+: now reaches K1.3
- net AIR+: now also J15.2 (Pin_2); no longer J15.1 (Pin_1)
- net OSC2: now reaches U1.8 (OSC2), Y1.1 (INPUT)
- net OSC1: now reaches U1.9 (OSC1), Y1.3 (OUTPUT)
- net at D2.2 (A), K1.1: now also Q2.3 (D)
- net PRECHARGE: now reaches K1.4
- net PRECHARGE: now also J14.2 (Pin_2); no longer J14.1 (Pin_1)
- net RtD_LED: now reaches J17.1 (Pin_1)
- net RtD_LED: now also Q4.3 (D)
- net *2 renamed *2/INT_A
- net +3V3 renamed +3.3V
- net ~{RESET} renamed RESET
- no-connect marks 12 -> 41
Other:
- note added: "+5V"
- note added: "Accel1"
- note added: "Accel2"
- note added: "Brake"
- note added: "CAN"
- note added: "Power"
- note added: "RESET"
- note added: "SCL/21"
- note added: "SDA/20"
- note added: "Shutdown Circuit"
- moved on the sheet: C2, D2, D3, J10, J11, J12, J13, J14, J15, J16, J17, J18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

Commit message: 基板配置まで
Connections:
- net *10: now also Q1.3 (D), R3.2; no longer J18.1 (Pin_1), R11.1
- net *11: now also J19.1 (Pin_1), R12.1; no longer Q1.3 (D), R3.2
- net *12: now also J18.1 (Pin_1), R11.1; no longer Q3.1 (G), R8.1
- net *13: now also Q4.1 (G), R9.1; no longer Q2.1 (G), R7.1
- net *3: now also Q3.1 (G), R8.1
- net *4: now also Q2.1 (G), R7.1
- net *7: no longer Q4.1 (G), R9.1
- net *8: no longer J19.1 (Pin_1), R12.1
- net CANH: now also J20.1 (Pin_1); no longer J20.2 (Pin_2)
- net CANL: now also J20.2 (Pin_2); no longer J20.1 (Pin_1)
Other:
- moved on the sheet: D2, D3, J14, J15, J16, J17, J18, J19, J20, K1, K2, Q2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

Commit message: パターン設計途中
Connections:
- net COIL1: now reaches D2.2 (A), K1.1, Q2.3 (D)
- net COIL2: now reaches D3.2 (A), K2.1, Q3.3 (D)
Changed lines of the file:
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@@
     (effects (font (size 1.27 1.27)) (justify right bottom))
+  )
+  (label "COIL2" (at 228.6 137.16 0) (fields_autoplaced)
+    (effects (font (size 1.27 1.27)) (justify left bottom))
   )
   (label "IOREF" (at 119.38 27.94 0) (fields_autoplaced)
@@
     (effects (font (size 1.27 1.27)) (justify right bottom))
   )
+  (label "COIL1" (at 195.58 119.38 0) (fields_autoplaced)
+    (effects (font (size 1.27 1.27)) (justify left bottom))
+  )
   (label "A7" (at 121.92 93.98 0) (fields_autoplaced)

Commit message: modify, finish, ver3
Connections:
- net +12V: now also D2.1 (K), D3.1 (K), K1.5, K2.5
- net SHUTDOWN_CIRCUIT: no longer D2.1 (K), D3.1 (K), K1.5, K2.5
Changed lines of the file:
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@@
   (junction (at 132.08 40.64) (diameter 1.016) (color 0 0 0 0)
   )
+  (junction (at 233.68 48.26) (diameter 0) (color 0 0 0 0)
+  )
   (junction (at 238.76 121.92) (diameter 0) (color 0 0 0 0)
   )
-  (junction (at 205.74 99.06) (diameter 0) (color 0 0 0 0)
-  )
-  (junction (at 233.68 48.26) (diameter 0) (color 0 0 0 0)
-  )
   (junction (at 238.76 137.16) (diameter 0) (color 0 0 0 0)
   )
@@
   (junction (at 88.9 43.18) (diameter 0) (color 0 0 0 0)
   )
+  (junction (at 246.38 81.28) (diameter 0) (color 0 0 0 0)
+  )
+  (junction (at 256.54 116.84) (diameter 0) (color 0 0 0 0)
+  )
   (junction (at 205.74 104.14) (diameter 0) (color 0 0 0 0)
-  )
-  (junction (at 246.38 81.28) (diameter 0) (color 0 0 0 0)
-  )
-  (junction (at 256.54 116.84) (diameter 0) (color 0 0 0 0)
   )
   (junction (at 205.74 134.62) (diameter 0) (color 0 0 0 0)
@@
     (stroke (width 0) (type default))
   )
-  (wire (pts (xy 205.74 93.98) (xy 205.74 99.06))
-    (stroke (width 0) (type default))
-  )
   (wire (pts (xy 248.92 33.02) (xy 259.08 33.02))
     (stroke (width 0) (type default))
@@
     (stroke (width 0) (type default))
   )
-  (wire (pts (xy 205.74 99.06) (xy 238.76 99.06))
-    (stroke (width 0) (type default))
-  )
   (wire (pts (xy 165.1 162.56) (xy 152.4 162.56))
     (stroke (width 0) (type default))
@@
     (stroke (width 0) (type default))
   )
-  (wire (pts (xy 205.74 99.06) (xy 205.74 104.14))
-    (stroke (width 0) (type default))
-  )
   (wire (pts (xy 241.3 58.42) (xy 233.68 58.42))
     (stroke (width 0) (type default))
@@
     (stroke (width 0) (type default))
   )
-  (wire (pts (xy 238.76 99.06) (xy 238.76 121.92))
-    (stroke (width 0) (type default))
-  )
   (wire (pts (xy 160.02 88.9) (xy 175.26 88.9))
     (stroke (width 0) (type solid))
@@
   (label "A12" (at 121.92 111.76 0) (fields_autoplaced)
     (effects (font (size 1.27 1.27)) (justify left bottom))
-  )
-  (global_label "SHUTDOWN_CIRCUIT" (shape input) (at 205.74 93.98 0) (fields_autoplaced)
-    (effects (font (size 1.27 1.27)) (justify left))
-    (property "Intersheetrefs" "${INTERSHEET_REFS}" (at 227.2467 93.98 0)
-      (effects (font (size 1.27 1.27)) (justify left) hide)
-    )
   )
   (global_label "SHUTDOWN_CIRCUIT" (shape input) (at 215.9 119.38 0) (fields_autoplaced)
@@
         (path "/e63e39d7-6ac0-4ffd-8aa3-1841a4541b55"
           (reference "R13") (unit 1)
+        )
+      )
+    )
+  )
+  (symbol (lib_id "power:+12V") (at 238.76 121.92 0) (unit 1)
+    (in_bom yes) (on_board yes) (dnp no) (fields_autoplaced)
+    (property "Reference" "#PWR037" (at 238.76 125.73 0)
+      (effects (font (size 1.27 1.27)) hide)
+    )
+    (property "Value" "+12V" (at 238.76 116.84 0)
+      (effects (font (size 1.27 1.27)))
+    )
+    (property "Footprint" "" (at 238.76 121.92 0)
+      (effects (font (size 1.27 1.27)) hide)
+    )
+    (property "Datasheet" "" (at 238.76 121.92 0)
+      (effects (font (size 1.27 1.27)) hide)
+    )
+    (pin "1")
+    (instances
+      (project "ECUShield_MEGA_ver1"
+        (path "/e63e39d7-6ac0-4ffd-8aa3-1841a4541b55"
+          (reference "#PWR037") (unit 1)
         )
       )
@@
         )
       )
+    )
+  )
+  (symbol (lib_id "power:+12V") (at 205.74 104.14 0) (unit 1)
+    (in_bom yes) (on_board yes) (dnp no) (fields_autoplaced)
+    (property "Reference" "#PWR036" (at 205.74 107.95 0)
+      (effects (font (size 1.27 1.27)) hide)
+    )
+    (property "Value" "+12V" (at 205.74 99.06 0)
+      (effects (font (size 1.27 1.27)))
+    )
+    (property "Footprint" "" (at 205.74 104.14 0)
+      (effects (font (size 1.27 1.27)) hide)
+    )
+    (property "Datasheet" "" (at 205.74 104.14 0)
+      (effects (font (size 1.27 1.27)) hide)
+    )
+    (pin "1")
+    (instances
+      (project "ECUShield_MEGA_ver1"
+        (path "/e63e39d7-6ac0-4ffd-8aa3-1841a4541b55"
+          (reference "#PWR036") (unit 1)
+        )
+      )

Commit message: 回路図修正, パターン再設計
Parts:
- removed J6: Conn_01x02_Pin, Connector_JST:JST_XH_B2B-XH-A_1x02_P2.50mm_Vertical, symbol Connector:Conn_01x02_Pin
- removed K2: G5Q-1, Relay_THT:Relay_SPDT_Omron-G5Q-1, symbol Relay:G5Q-1
- removed Q1: MTN2306AN3, Package_TO_SOT_SMD:TSOT-23, symbol Device:Q_NMOS_GSD
- removed U1: MCP2515-xST, Package_SO:TSSOP-20_4.4x6.5mm_P0.65mm, symbol Interface_CAN_LIN:MCP2515-xST
- added C2, C3, C4: 0.1u, Capacitor_SMD:C_0603_1608Metric, symbol Device:C
- added D4: 1S953, Diode_THT:D_DO-35_SOD27_P7.62mm_Horizontal, symbol Device:D
- added J13: Conn_01x02_Pin, Connector_JST:JST_XH_B2B-XH-A_1x02_P2.50mm_Vertical, symbol Connector:Conn_01x02_Pin
- added J6: Conn_01x03_Pin, Connector_JST:JST_XH_B3B-XH-A_1x03_P2.50mm_Vertical, symbol Connector:Conn_01x03_Pin
- added JP1, JP2: SolderJumper_2_Open, Jumper:SolderJumper-2_P1.3mm_Open_RoundedPad1.0x1.5mm, symbol Jumper:SolderJumper_2_Open
- added K1, K3: G5Q-1A, Relay_THT:Relay_SPST_Omron-G5Q-1A, symbol Relay:G5Q-1A
- added R3: 100k, Resistor_SMD:R_0603_1608Metric, symbol Device:R
- added U1: MCP2515-xSO, Package_SO:SOIC-18W_7.5x11.6mm_P1.27mm, symbol Interface_CAN_LIN:MCP2515-xSO
- R1: value 10k -> 100k; footprint Resistor_SMD:R_0805_2012Metric -> Resistor_SMD:R_0603_1608Metric
- R2: value 1M -> 100k
- renumbered C2 to C5, J13 to J14, J17 to J15, J18 to J16, J19 to J17, J14 to J18, J15 to J19, J16 to J20, J20 to J21, K1 to K2, Q2 to Q1, Q3 to Q2, Q4 to Q3, R9 to R10, R10 to R11, R11 to R12, R12 to R13, R13 to R14, R3 to R4, R4 to R5, R5 to R6, R6 to R7, R7 to R8, R8 to R9
Connections:
- net *10: no longer R4.2
- net *2/INT_A: now also U1.12 (~{INT})
- net *4: now also JP2.2 (B); no longer Q1.1 (G), R8.1
- net *5: now also JP1.2 (B)
- net *6: now also Q1.1 (G), R8.1
- net *7: now also J13.2 (Pin_2)
- net *8: now also R4.1, K1.2
- net *9/CS_A: now also U1.16 (~{CS})
- net +12V: now also K3.5
- net +5V: now also J6.1 (Pin_1), K1.3, U1.18 (VDD); no longer R1.1, R4.1
- net A0: now also R1.1, C2.1
- net A1: now also R2.1, C3.1
- net A2: now also C4.1, J6.2 (Pin_2), R3.1; no longer R1.2
- net AIR-: now also K3.3
- net COIL2: now also K3.1
- net GND: now also R1.2, R4.2, C2.2, C3.2, C4.2, D4.2 (A), J13.1 (Pin_1), J6.3 (Pin_3), K1.1, R3.2, U1.9 (VSS)
- net MISO_A: now also U1.15 (SO)
- net MOSI_A: now also U1.14 (SI)
- net OSC1: now also U1.8 (OSC1)
- net OSC2: now also U1.7 (OSC2)
- net RXCAN: now also JP1.1 (A), U1.2 (RXCAN)
- net SCK_A: now also U1.13 (SCK)
- net SHUTDOWN_CIRCUIT: now also D4.1 (K), K1.5, K3.2; no longer R2.1
- net TXCAN: now also JP2.1 (A), U1.1 (TXCAN)
- net at R5.2: now also U1.17 (~{RESET})
- no-connect marks 41 -> 37
Other:
- note added: "Sound"
- moved on the sheet: C5, J10, J2, J3, J4, J5, J7, R4

Commit message: 修正版寝かせ
Parts:
- added J22: Conn_01x02_Pin, Connector_JST:JST_XH_B2B-XH-A_1x02_P2.50mm_Vertical, symbol Connector:Conn_01x02_Pin
Connections:
- net *10: now also J22.2 (Pin_2)
- net GND: now also J22.1 (Pin_1)
- no-connect marks 37 -> 36
Other:
- note removed: "Sound"
Changed lines of the file:
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@@
   (no_connect (at 172.72 114.3))
   (no_connect (at 172.72 111.76))
-  (no_connect (at 172.72 48.26))
   (no_connect (at 50.8 139.7))
   (no_connect (at 91.44 182.88))
@@
     (stroke (width 0) (type default))
   )
+  (wire (pts (xy 198.12 53.34) (xy 190.5 53.34))
+    (stroke (width 0) (type default))
+  )
   (wire (pts (xy 60.96 165.1) (xy 20.32 165.1))
     (stroke (width 0) (type default))
@@
     (stroke (width 0) (type default))
   )
+  (wire (pts (xy 190.5 53.34) (xy 190.5 48.26))
+    (stroke (width 0) (type default))
+  )
   (wire (pts (xy 48.26 104.14) (xy 48.26 106.68))
     (stroke (width 0) (type default))
@@
     (stroke (width 0) (type default))
   )
-  (wire (pts (xy 160.02 48.26) (xy 172.72 48.26))
-    (stroke (width 0) (type default))
-  )
   (wire (pts (xy 160.02 114.3) (xy 172.72 114.3))
     (stroke (width 0) (type solid))
@@
     (stroke (width 0) (type solid))
   )
+  (wire (pts (xy 160.02 48.26) (xy 190.5 48.26))
+    (stroke (width 0) (type default))
+  )
   (wire (pts (xy 60.96 160.02) (xy 17.78 160.02))
     (stroke (width 0) (type default))
@@
     (effects (font (size 1.27 1.27)) (justify left bottom))
   )
-  (text "Sound" (at 204.47 74.93 0)
-    (effects (font (size 1.27 1.27)) (justify left bottom))
-  )
   (text "AIR-" (at 266.7 113.03 0)
     (effects (font (size 1.27 1.27)) (justify left bottom))
@@
     )
   )
+  (symbol (lib_id "Connector:Conn_01x02_Pin") (at 203.2 55.88 180) (unit 1)
+    (in_bom yes) (on_board yes) (dnp no) (fields_autoplaced)
+    (property "Reference" "J22" (at 204.47 53.34 0)
+      (effects (font (size 1.27 1.27)) (justify right))
+    )
+    (property "Value" "Conn_01x02_Pin" (at 204.47 55.88 0)
+      (effects (font (size 1.27 1.27)) (justify right))
+    )
+    (property "Footprint" "Connector_JST:JST_XH_B2B-XH-A_1x02_P2.50mm_Vertical" (at 203.2 55.88 0)
+      (effects (font (size 1.27 1.27)) hide)
+    )
+    (property "Datasheet" "~" (at 203.2 55.88 0)
+      (effects (font (size 1.27 1.27)) hide)
+    )
+    (pin "1")
+    (pin "2")
+    (instances
+      (project "ECUShield_MEGA_ver1"
+        (path "/e63e39d7-6ac0-4ffd-8aa3-1841a4541b55"
+          (reference "J22") (unit 1)
+        )
+      )
+    )
+  )
   (symbol (lib_id "power:+12V") (at 256.54 40.64 0) (unit 1)
     (in_bom yes) (on_board yes) (dnp no) (fields_autoplaced)
@@
         )
       )
+    )
+  )
+  (symbol (lib_id "power:GND") (at 198.12 55.88 0) (unit 1)
+    (in_bom yes) (on_board yes) (dnp no)
+    (property "Reference" "#PWR042" (at 198.12 62.23 0)
+      (effects (font (size 1.27 1.27)) hide)
+    )
+    (property "Value" "GND" (at 198.12 59.69 0)
+      (effects (font (size 1.27 1.27)))
+    )
+    (property "Footprint" "" (at 198.12 55.88 0)
+      (effects (font (size 1.27 1.27)))
+    )
+    (property "Datasheet" "" (at 198.12 55.88 0)
+      (effects (font (size 1.27 1.27)))
+    )
+    (pin "1")
+    (instances
+      (project "ECUShield_MEGA_ver1"
+        (path "/e63e39d7-6ac0-4ffd-8aa3-1841a4541b55"
+          (reference "#PWR042") (unit 1)
+        )
+      )
