File: AMS_Temp_Master/AMS_Temp_Master.kicad_sch (KiCad schematic)
At the start: 37 parts, among them J1 Conn_01x10_Socket, J2 Conn_01x02_Pin, J3 Conn_01x02_Pin, J4 Conn_01x04_Pin, J5 Conn_01x02_Pin, Q1 AO3401A, U1 ATmega328P-A, U2 MCP2515-xSO, U3 MCP2551-I-SN, U4 LD1117S50TR_SOT223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

Commit message: 10k抵抗フットプリント修正2012
Parts:
- R10, R3, R7, R9: footprint Resistor_SMD:R_0603_1608Metric -> Resistor_SMD:R_0805_2012Metric
Changed lines of the file:
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@@
       (effects (font (size 1.27 1.27)) (justify left))
     )
-    (property "Footprint" "Resistor_SMD:R_0603_1608Metric" (at 234.442 120.65 90)
+    (property "Footprint" "Resistor_SMD:R_0805_2012Metric" (at 234.442 120.65 90)
       (effects (font (size 1.27 1.27)) hide)
     )
@@
       (effects (font (size 1.27 1.27)) (justify left))
     )
-    (property "Footprint" "Resistor_SMD:R_0603_1608Metric" (at 173.482 77.47 90)
+    (property "Footprint" "Resistor_SMD:R_0805_2012Metric" (at 173.482 77.47 90)
       (effects (font (size 1.27 1.27)) hide)
     )
@@
       (effects (font (size 1.27 1.27)) (justify left))
     )
-    (property "Footprint" "Resistor_SMD:R_0603_1608Metric" (at 226.822 36.83 90)
+    (property "Footprint" "Resistor_SMD:R_0805_2012Metric" (at 226.822 36.83 90)
       (effects (font (size 1.27 1.27)) hide)
     )
@@
       (effects (font (size 1.27 1.27)) (justify left))
     )
-    (property "Footprint" "Resistor_SMD:R_0603_1608Metric" (at 115.062 123.19 90)
-      (effects (font (size 1.27 1.27)) hide)
-    )
+    (property "Footprint" "Resistor_SMD:R_0805_2012Metric" (at 115.062 123.19 90)
+      (effects (font (size 1.27 1.27)) hide)
+    )

Commit message: 回路図微修正
Parts:
- C10: value 470u -> 47u
Changed lines of the file:
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@@
       (effects (font (size 1.27 1.27)) (justify left))
     )
-    (property "Value" "470u" (at 222.25 30.226 0)
+    (property "Value" "47u" (at 222.25 30.226 0)
       (effects (font (size 1.27 1.27)) (justify left))
     )
